File: eagle/packmonitor/packmonitor.brd (EAGLE design)
At the start: 61 x 18 mm, 32 parts, among them IC1 24C64, IC2 TCA4311A, IC3 AP2411, IC4 ACS712

Commit message: made some good progress on the board this afternoon!
Parts:
- removed BATIN, BATOUT: (no value), SparkFun-Connectors:SCREWTERMINAL-3.5MM-2
- removed C1, C4: 100n, rcl:C0603
- removed U$8: MOSFET-PCHANNEL-SOIC8SOIC8, SparkFun-DiscreteSemi:SO08
- added CACS, CTCA, CVCC: 100n, rcl:C0603
- added GROUND, OUT: (no value), SparkFun-Connectors:SCREWTERMINAL-3.5MM-2
- added Q1: PCHAN, SparkFun-DiscreteSemi:SO08
- added RG-PU: 10K, rcl:R0603
- added RGATE: 470R, rcl:R0603
- RBUS1, RBUS2, RPACK1, RPACK2, TR1, TR2, TR3: device rcl:R0603 -> rcl:R0805
- moved RPACK2 15.1 mm to (55.6, 3.05), turned to 90 degrees
- moved RPACK1 9.57 mm to (55.6, 8.64), turned to 90 degrees
- moved IC4 1.27 mm to (49.5, 10.2), turned to 180 degrees
- moved TR3 0.25 mm to (49.3, 5.08)
- renumbered C2 to CAVCC, C3 to CEEP, C5 to CAP1, C6 to CAP2, C7 to CAP3
Connections:
- removed net N$1: IC4.3, IC4.4
- new net GATE: Q1.4, RG-PU.1, RGATE.1
- new net GATEDRV: A1.24, RGATE.2
- new net MVAOUT: A1.23, IC4.7
- new net P+IN: IC4.3, IC4.4, Q1.1, Q1.2, Q1.3
- new net P+OUT: OUT.1, Q1.5, Q1.6, Q1.7, Q1.8
- net GND: now also CACS.2, CTCA.2, CVCC.2, GROUND.1, GROUND.2, IC4.5; no longer BATIN.2, BATOUT.1, C1.2, C4.2
- net TS0: now also A1.14; no longer A1.16
- net TS2: now also A1.16; no longer A1.14
- net VBAT: now also A1.17; no longer A1.24
- net VCC: now also CACS.1, CTCA.1, CVCC.1, IC4.8; no longer C1.1, C4.1
- net VPACK: now also OUT.2, RG-PU.2; no longer BATIN.1
Routing:
- net VCC: track 35.9 -> 92.7 mm, vias 3 -> 4
- net TS2: track 0.00 -> 19.8 mm
- net MVAOUT: track 0.00 -> 19.5 mm
- net VBAT: track 7.79 -> 24.2 mm, vias 0 -> 1
- net TS1: track 0.00 -> 16.4 mm
- net GATE: track 0.00 -> 14.3 mm, vias 0 -> 2
- net TS0: track 0.00 -> 12.3 mm
- net UPDI: track 0.00 -> 5.90 mm
- net VPACK: track 0.00 -> 3.39 mm, vias 0 -> 11
- net GATEDRV: track 0.00 -> 2.84 mm
- net GND: track 12.4 -> 14.3 mm, vias 2 -> 7
- added copper zone on layer 1, net GND
- added copper zone on layer 1, net P+IN
- added copper zone on layer 16, net P+IN
- added copper zone on layer 1, net P+OUT
- added copper zone on layer 16, net P+OUT
- added copper zone on layer 16, net VPACK
Other:
- board size 61 x 18 mm -> 62.3 x 18 mm
