File: eagle/packmonitor/packmonitor.sch (EAGLE design)
At the start: 12 parts, among them IC2 24C64

Commit message: making good progress on schematic and board layout
Parts:
- removed J1: (no value), SparkFun-Connectors:M03LOCK_LONGPADS
- added C4, C5, C6: 100n, rcl:C-USC0603
- added C7: 120u, rcl:C-USC1206
- added IC1: 24C64, microchip:24C04CSN
- added IC3: AP2411, ti-special:TPS2041BD
- added R1, R3, R4: 10K, rcl:R-US_R0603
- added R2: (no value), rcl:R-US_R0603
- added UPDI: (no value), SparkFun-Connectors:M03LOCK_LONGPADS
- A1: value ATMEGA4808-TQFN32A -> ATMEGA4808
- C1, C2, C3: value 100u -> 100n
- IC2: value 24C64 -> TCA4311A; device microchip:24C04CSN -> NXP_By_element14_Batch_1:PCA9511AD,118
- renumbered J2 to BATIN, J3 to BATOUT
Connections:
- removed net N$2: A1.UPDI, J1.2
- new net BUSREADY: IC2.READY, R2.1
- new net ENBUSPWR: IC3./EN, R3.1
- new net N$3: HOSTCON.2, IC2.SDAIN
- new net N$4: HOSTCON.4, IC2.SCLIN
- new net N$6: IC2.ENABLE, R1.1
- new net PWRFAULT: IC3./OC, R4.1
- new net UPDI: A1.UPDI, UPDI.2
- new net VCCIO: C5.1, HOSTCON.6, IC3.IN1, IC3.IN2, R1.2, R3.2
- net A0: now also IC1.A0; no longer IC2.A0
- net A1: now also IC1.A1; no longer IC2.A1
- net A2: now also IC1.A2; no longer IC2.A2
- net GND: now also BATIN.2, BATOUT.1, C4.2, C5.2, C6.2, C7.2, IC1.GND, IC1.WP, IC3.GND, UPDI.1; no longer IC2.WP, J1.1
- net SCL: now also IC1.SCL, IC2.SCLOUT; no longer HOSTCON.2, IC2.SCL
- net SDA: now also IC1.SDA, IC2.SDAOUT; no longer HOSTCON.4, IC2.SDA
- net VCC: now also C4.1, C6.1, C7.1, IC1.VCC, IC3.OUT1, IC3.OUT2, IC3.OUT3, R2.2, R4.2, UPDI.3; no longer HOSTCON.6, J1.3
Other:
- moved on the sheet: HOSTCON

Commit message: making progress slowly
Parts:
- removed HOSTCON: (no value), SparkFun-Connectors:M06RA
- added IC4: ACS712, SparkFun-AnalogIC:ACS712
- added RBUS1, RBUS2, TR1, TR2, TR3: 50K, rcl:R-US_R0603
- added RPACK1: 120K, rcl:R-US_R0603
- added RPACK2: 30K, rcl:R-US_R0603
- added THERM: JST-XH-06-PIN-ROUND-PAD, Rembrandt Electronics - JST XH Connectors v1-0:JST-XH-06-PIN-ROUND-PAD
- added U$8: MOSFET-PCHANNEL-SOIC8SOIC8, SparkFun-DiscreteSemi:MOSFET-PCHANNEL-SOIC8SOIC8
- added X1: JST-XH-06-PIN-LONG-PAD, Rembrandt Electronics - JST XH Connectors v1-0:JST-XH-06-PIN-LONG-PAD
- JP1: value A) -> A1
- UPDI: device SparkFun-Connectors:M03LOCK_LONGPADS -> SparkFun-Connectors:M03PTH
Connections:
- new net N$1: IC4.IP-@3, IC4.IP-@4
- new net TS0: A1.PD6(A6/AIN6/AC-P2/TCA0), THERM-2.S, TR1.2
- new net TS1: A1.PD5(A5/AIN5/AC-N1/TCA0), THERM-4.S, TR2.2
- new net TS2: A1.PD4(A4/AIN4/AC-P1/TCA0), THERM-6.S, TR3.2
- new net VBAT: A1.PF4(A10/AIN14/TXD2), RPACK1.1, RPACK2.2
- new net VBUS: A1.PD0(A0/AIN0/2-IN0/TCA0), RBUS1.1, RBUS2.2
- new net VPACK: BATIN.1, IC4.IP+@1, IC4.IP+@2, RPACK1.2
- net GND: now also RBUS2.1, RPACK2.1, TR1.1, TR2.1, TR3.1, X1-2.S, X1-4.S, X1-6.S; no longer HOSTCON.1, HOSTCON.3, HOSTCON.5
- net N$3: now also X1-5.S; no longer HOSTCON.2
- net N$4: now also X1-3.S; no longer HOSTCON.4
- net VCC: now also THERM-1.S, THERM-3.S, THERM-5.S
- net VCCIO: now also RBUS1.2, X1-1.S; no longer HOSTCON.6
Other:
- moved on the sheet: BATIN, BATOUT
