File: eagle/packmonitor/packmonitor.sch (EAGLE design)
At the start: 32 parts, among them IC1 24C64, IC2 TCA4311A, IC3 AP2411, IC4 ACS712, X1 JST-XH-06-PIN-LONG-PAD

Commit message: made some good progress on the board this afternoon!
Parts:
- removed BATIN, BATOUT: (no value), SparkFun-Connectors:M023.5MM
- removed U$8: MOSFET-PCHANNEL-SOIC8SOIC8, SparkFun-DiscreteSemi:MOSFET-PCHANNEL-SOIC8SOIC8
- added CACS: 100n, rcl:C-USC0603
- added GROUND, OUT: (no value), SparkFun-Connectors:M023.5MM
- added Q1: PCHAN, SparkFun-DiscreteSemi:MOSFET-PCHANNEL-SOIC8SOIC8
- added RG-PU: 10K, rcl:R-US_R0603
- added RGATE: 470R, rcl:R-US_R0603
- RBUS1, RBUS2, RPACK1, RPACK2, TR1, TR2, TR3: device rcl:R-US_R0603 -> rcl:R-US_R0805
- renumbered C1 to CVCC, C2 to CAVCC, C3 to CEEP, C4 to CTCA, C5 to CAP1, C6 to CAP2, C7 to CAP3
Connections:
- removed net N$1: IC4.IP-@3, IC4.IP-@4
- new net GATE: Q1.G, RG-PU.1, RGATE.1
- new net GATEDRV: A1.PF4(A10/AIN14/TXD2), RGATE.2
- new net MVAOUT: A1.PF3(A9/AIN13/3-OUT), IC4.VOUT
- new net P+IN: IC4.IP-@3, IC4.IP-@4, Q1.S@1, Q1.S@2, Q1.S@3
- new net P+OUT: OUT.1, Q1.D@1, Q1.D@2, Q1.D@3, Q1.D@4
- net GND: now also CACS.2, GROUND.1, GROUND.2, IC4.GND; no longer BATIN.2, BATOUT.1
- net TS0: now also A1.PD4(A4/AIN4/AC-P1/TCA0); no longer A1.PD6(A6/AIN6/AC-P2/TCA0)
- net TS2: now also A1.PD6(A6/AIN6/AC-P2/TCA0); no longer A1.PD4(A4/AIN4/AC-P1/TCA0)
- net VBAT: now also A1.PD7(A7/AIN7/AC-N2/AREF); no longer A1.PF4(A10/AIN14/TXD2)
- net VCC: now also CACS.1, IC4.VCC
- net VPACK: now also OUT.2, RG-PU.2; no longer BATIN.1
Other:
- moved on the sheet: IC4, RPACK1, RPACK2, THERM-1, THERM-2, THERM-3, THERM-4, THERM-5, THERM-6, TR1, TR2, TR3
